File: Martin-V-USB_Mame_Panel_Atmega8ISP-V20f.brd (EAGLE design)
At the start: 50 x 50 mm, 20 parts, among them IC1 MEGA8-P, IC2 LD117ADT33TR, Q1 12MHz, X1 USB

Commit message: New Board Revision
Parts:
- added GND: (no value), con-lstb:MA07-1
- added VCC: (no value), con-lstb:MA06-1
- moved C2 12.5 mm to (16.5, 22.9)
- moved C1 6.48 mm to (16.5, 17.8)
- moved R4 6.35 mm to (19.1, 8.89)
- moved R1 6.35 mm to (19.1, 12.7)
- moved D1 3.81 mm to (26.7, 14.0)
- moved R5 2.84 mm to (8.89, 17.8)
- moved C3 2.84 mm to (24.1, 22.9), turned to 180 degrees
- moved R3 1.80 mm to (11.4, 17.8)
- moved SV1 1.27 mm to (5.08, 33.0)
Connections:
- net +5V: now also VCC.1, VCC.2, VCC.3, VCC.4, VCC.5, VCC.6
- net GND: now also GND.1, GND.2, GND.3, GND.4, GND.5, GND.6, GND.7
Routing:
- net GND: track 135.8 -> 0.00 mm
- net +5V: track 49.7 -> 80.0 mm
- net COINTRIGGER: track 53.1 -> 32.4 mm, vias 1 -> 0
- net JOY1BUTTON3: track 34.7 -> 14.6 mm
- net JOY1UP: track 61.4 -> 43.5 mm, vias 2 -> 0
- net JOY2START: track 59.4 -> 46.2 mm
- net +3V3: track 91.9 -> 79.9 mm
- net N$2: track 30.5 -> 19.4 mm
- net JOY2LEFT: track 41.8 -> 31.0 mm, vias 1 -> 0
- net JOY1BUTTON1: track 24.7 -> 14.6 mm
- net N$4: track 47.1 -> 37.6 mm
- net JOY1LEFT: track 16.8 -> 25.7 mm, vias 1 -> 0
- net JOY2UP: track 28.5 -> 19.7 mm
- net JOY2BUTTON3: track 28.0 -> 36.2 mm, vias 1 -> 0
- net N$1: track 27.4 -> 19.3 mm
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- added copper zone on layer 1, net GND
- added copper zone on layer 16, net GND
- removed copper zone on layer 16, net N$6
- removed copper zone on layer 1, net N$7
