File: Martin-V-USB_Mame_Panel_Atmega8ISP-V20f.sch (EAGLE design)
At the start: 17 parts, among them IC1 MEGA8-P, IC2 LD117ADT33TR, Q1 12MHz, X1 USB

Commit message: New Board Revision
Parts:
- added GND: (no value), con-lstb:MA07-1
- added VCC: (no value), con-lstb:MA06-1
Connections:
- net +5V: now also VCC.1, VCC.2, VCC.3, VCC.4, VCC.5, VCC.6
- net GND: now also GND.1, GND.2, GND.3, GND.4, GND.5, GND.6, GND.7
Changed lines of the file:
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@@
 </variantdefs>
 <classes>
-<class number="0" name="default" width="0" drill="0">
+<class number="0" name="default" width="0.254" drill="0">
+</class>
+<class number="1" name="power" width="0.8128" drill="0">
 </class>
 </classes>
@@
 <part name="JOY1+2" library="con-lstb" deviceset="MA10-2W" device=""/>
 <part name="GND2" library="supply1" deviceset="GND" device=""/>
+<part name="VCC" library="con-lstb" deviceset="MA06-1" device=""/>
+<part name="GND" library="con-lstb" deviceset="MA07-1" device=""/>
+<part name="GND10" library="supply1" deviceset="GND" device=""/>
+<part name="P+2" library="supply1" deviceset="+5V" device=""/>
 </parts>
 <sheets>
@@
 <instance part="JOY1+2" gate="1" x="190.5" y="58.42"/>
 <instance part="GND2" gate="1" x="190.5" y="35.56"/>
+<instance part="VCC" gate="1" x="180.34" y="17.78" rot="R270"/>
+<instance part="GND" gate="1" x="205.74" y="17.78" rot="R270"/>
+<instance part="GND10" gate="1" x="205.74" y="0"/>
+<instance part="P+2" gate="1" x="190.5" y="0" rot="R270"/>
 </instances>
 <busses>
@@
 </segment>
 </net>
-<net name="GND" class="0">
+<net name="GND" class="1">
 <segment>
 <wire x1="129.54" y1="63.5" x2="129.54" y2="66.04" width="0.1524" layer="91"/>
@@
 <wire x1="190.5" y1="40.64" x2="190.5" y2="38.1" width="0.1524" layer="91"/>
 <junction x="190.5" y="40.64"/>
+</segment>
+<segment>
+<pinref part="GND" gate="1" pin="4"/>
+<pinref part="GND10" gate="1" pin="GND"/>
+<wire x1="205.74" y1="10.16" x2="205.74" y2="5.08" width="0.1524" layer="91"/>
+<pinref part="GND" gate="1" pin="1"/>
+<wire x1="205.74" y1="5.08" x2="205.74" y2="2.54" width="0.1524" layer="91"/>
+<wire x1="198.12" y1="10.16" x2="198.12" y2="5.08" width="0.1524" layer="91"/>
+<wire x1="198.12" y1="5.08" x2="200.66" y2="5.08" width="0.1524" layer="91"/>
+<junction x="205.74" y="5.08"/>
+<pinref part="GND" gate="1" pin="2"/>
+<wire x1="200.66" y1="5.08" x2="203.2" y2="5.08" width="0.1524" layer="91"/>
+<wire x1="203.2" y1="5.08" x2="205.74" y2="5.08" width="0.1524" layer="91"/>
+<wire x1="200.66" y1="10.16" x2="200.66" y2="5.08" width="0.1524" layer="91"/>
+<junction x="200.66" y="5.08"/>
+<pinref part="GND" gate="1" pin="3"/>
+<wire x1="203.2" y1="10.16" x2="203.2" y2="5.08" width="0.1524" layer="91"/>
+<junction x="203.2" y="5.08"/>
+<wire x1="205.74" y1="5.08" x2="208.28" y2="5.08" width="0.1524" layer="91"/>
+<pinref part="GND" gate="1" pin="7"/>
+<wire x1="208.28" y1="5.08" x2="210.82" y2="5.08" width="0.1524" layer="91"/>
+<wire x1="210.82" y1="5.08" x2="213.36" y2="5.08" width="0.1524" layer="91"/>
+<wire x1="213.36" y1="5.08" x2="213.36" y2="10.16" width="0.1524" layer="91"/>
+<pinref part="GND" gate="1" pin="6"/>
+<wire x1="210.82" y1="10.16" x2="210.82" y2="5.08" width="0.1524" layer="91"/>
+<junction x="210.82" y="5.08"/>
+<pinref part="GND" gate="1" pin="5"/>
+<wire x1="208.28" y1="10.16" x2="208.28" y2="5.08" width="0.1524" layer="91"/>
+<junction x="208.28" y="5.08"/>
 </segment>
 </net>
@@
 </segment>
 </net>
-<net name="+5V" class="0">
+<net name="+5V" class="1">
 <segment>
 <wire x1="152.4" y1="20.32" x2="152.4" y2="81.28" width="0.1524" layer="91"/>
@@
 <pinref part="D1" gate="G$1" pin="C"/>
 </segment>
+<segment>
+<pinref part="VCC" gate="1" pin="1"/>
+<wire x1="172.72" y1="10.16" x2="172.72" y2="0" width="0.1524" layer="91"/>
+<pinref part="P+2" gate="1" pin="+5V"/>
+<wire x1="172.72" y1="0" x2="175.26" y2="0" width="0.1524" layer="91"/>
+<pinref part="VCC" gate="1" pin="2"/>
+<wire x1="175.26" y1="0" x2="177.8" y2="0" width="0.1524" layer="91"/>
+<wire x1="177.8" y1="0" x2="180.34" y2="0" width="0.1524" layer="91"/>
+<wire x1="180.34" y1="0" x2="182.88" y2="0" width="0.1524" layer="91"/>
+<wire x1="182.88" y1="0" x2="185.42" y2="0" width="0.1524" layer="91"/>
+<wire x1="185.42" y1="0" x2="187.96" y2="0" width="0.1524" layer="91"/>
+<wire x1="175.26" y1="10.16" x2="175.26" y2="0" width="0.1524" layer="91"/>
+<junction x="175.26" y="0"/>
+<pinref part="VCC" gate="1" pin="3"/>
+<wire x1="177.8" y1="10.16" x2="177.8" y2="0" width="0.1524" layer="91"/>
+<junction x="177.8" y="0"/>
+<pinref part="VCC" gate="1" pin="4"/>
+<wire x1="180.34" y1="10.16" x2="180.34" y2="0" width="0.1524" layer="91"/>
+<junction x="180.34" y="0"/>
+<pinref part="VCC" gate="1" pin="5"/>
+<wire x1="182.88" y1="10.16" x2="182.88" y2="0" width="0.1524" layer="91"/>
+<junction x="182.88" y="0"/>
+<pinref part="VCC" gate="1" pin="6"/>
+<wire x1="185.42" y1="10.16" x2="185.42" y2="0" width="0.1524" layer="91"/>
+<junction x="185.42" y="0"/>
+</segment>
 </net>
 <net name="JOY1RIGHT" class="0">
@@
 </segment>
 </net>
-<net name="+3V3" class="0">
+<net name="+3V3" class="1">
 <segment>
 <wire x1="33.02" y1="43.18" x2="33.02" y2="40.64" width="0.1524" layer="91"/>
