File: Martin-V-USB_Mame_Panel_Atmega8ISP-V30-final.sch (EAGLE design)
At the start: 19 parts, among them IC1 MEGA8-P, IC2 LD117ADT33TR, Q1 12MHz, X1 USB

Commit message: v3
Parts:
- removed VCC: (no value), con-lstb:MA06-1
- GND: device con-lstb:MA07-1 -> con-lstb:MA04-1
- JOY1+2: device con-lstb:MA10-2W -> con-lstb:MA10-2
Connections:
- net +5V: no longer VCC.1, VCC.2, VCC.3, VCC.4, VCC.5, VCC.6
- net COINTRIGGER: now also JOY1+2.2; no longer JOY1+2.4
- net GND: now also JOY1+2.20; no longer GND.5, GND.6, GND.7, JOY1+2.2
- net JOY1BUTTON1: now also JOY1+2.8; no longer JOY1+2.12
- net JOY1BUTTON2: now also JOY1+2.7; no longer JOY1+2.10
- net JOY1BUTTON3: now also JOY1+2.9; no longer JOY1+2.8
- net JOY1DOWN: now also JOY1+2.3; no longer JOY1+2.20
- net JOY1LEFT: now also JOY1+2.6; no longer JOY1+2.16
- net JOY1RIGHT: now also JOY1+2.5; no longer JOY1+2.14
- net JOY1START: now also JOY1+2.10; no longer JOY1+2.6
- net JOY1UP: now also JOY1+2.4; no longer JOY1+2.18
- net JOY2BUTTON1: now also JOY1+2.13; no longer JOY1+2.11
- net JOY2BUTTON2: now also JOY1+2.14; no longer JOY1+2.9
- net JOY2BUTTON3: now also JOY1+2.11; no longer JOY1+2.7
- net JOY2DOWN: now also JOY1+2.17; no longer JOY1+2.19
- net JOY2LEFT: now also JOY1+2.16; no longer JOY1+2.15
- net JOY2RIGHT: now also JOY1+2.15; no longer JOY1+2.13
- net JOY2START: now also JOY1+2.12; no longer JOY1+2.5
- net JOY2UP: now also JOY1+2.18; no longer JOY1+2.17
- net SHIFTSWITCH: now also JOY1+2.19; no longer JOY1+2.3
